Commit message: [jvrc1.urdf] change gripper joint limits. change multiplier of gripper mimic joints.

File: jvrc_description/urdf/jvrc1.urdf (robot description, URDF)
Before this commit: robot jvrc1, 60 links, 59 joints
Joints:
- joint L_LINDEX: mimic joint=L_UTHUMB multiplier=-2 offset=0 -> joint=L_UTHUMB multiplier=-3 offset=0
- joint L_LLITTLE: mimic joint=L_UTHUMB multiplier=-2 offset=0 -> joint=L_UTHUMB multiplier=-3 offset=0
- joint L_LTHUMB: mimic joint=L_UTHUMB multiplier=2 offset=0 -> joint=L_UTHUMB multiplier=3 offset=0
- joint L_UINDEX: mimic joint=L_UTHUMB multiplier=-2 offset=0 -> joint=L_UTHUMB multiplier=-1 offset=0
- joint L_ULITTLE: mimic joint=L_UTHUMB multiplier=-2 offset=0 -> joint=L_UTHUMB multiplier=-1 offset=0
- joint L_UTHUMB: limit lower=-0.0 upper=0.785398163397 effort=100.0 velocity=6.80678 -> lower=-0.785398163397 upper=0.785398163397 effort=100.0 velocity=6.80678
- joint R_LINDEX: mimic joint=R_UTHUMB multiplier=-2 offset=0 -> joint=R_UTHUMB multiplier=-3 offset=0
- joint R_LLITTLE: mimic joint=R_UTHUMB multiplier=-2 offset=0 -> joint=R_UTHUMB multiplier=-3 offset=0
- joint R_LTHUMB: mimic joint=R_UTHUMB multiplier=2 offset=0 -> joint=R_UTHUMB multiplier=3 offset=0
- joint R_UINDEX: mimic joint=R_UTHUMB multiplier=-2 offset=0 -> joint=R_UTHUMB multiplier=-1 offset=0
- joint R_ULITTLE: mimic joint=R_UTHUMB multiplier=-2 offset=0 -> joint=R_UTHUMB multiplier=-1 offset=0
- joint R_UTHUMB: limit lower=-0.785398163397 upper=0.0 effort=100.0 velocity=6.80678 -> lower=-0.785398163397 upper=0.785398163397 effort=100.0 velocity=6.80678

Commit message: [jvrc1.urdf] Widen the width of the grippers.
This change corresponds to the change in https://github.com/jrl-umi3218/mc_openrtm/commit/48fc905eaddd2995bf639eca26b77e7be2d8ff28

File: jvrc_description/urdf/jvrc1.urdf (robot description, URDF)
Before this commit: robot jvrc1, 60 links, 59 joints
Joints:
- joint L_UINDEX: origin xyz=0.025 0.006 -0.102 rpy=0.0 -0.0 0.0 -> xyz=0.025 0.016 -0.084 rpy=0.0 -0.0 0.0
- joint L_ULITTLE: origin xyz=-0.025 0.006 -0.102 rpy=0.0 -0.0 0.0 -> xyz=-0.025 0.016 -0.084 rpy=0.0 -0.0 0.0
- joint L_UTHUMB: origin xyz=0.0 -0.023 -0.084 rpy=0.0 -0.0 0.0 -> xyz=0.0 -0.033 -0.084 rpy=0.0 -0.0 0.0
- joint R_UINDEX: origin xyz=0.025 -0.006 -0.102 rpy=0.0 -0.0 0.0 -> xyz=0.025 -0.016 -0.084 rpy=0.0 -0.0 0.0
- joint R_ULITTLE: origin xyz=-0.025 -0.006 -0.102 rpy=0.0 -0.0 0.0 -> xyz=-0.025 -0.016 -0.084 rpy=0.0 -0.0 0.0
- joint R_UTHUMB: origin xyz=0.0 0.023 -0.084 rpy=0.0 -0.0 0.0 -> xyz=0.0 0.033 -0.084 rpy=0.0 -0.0 0.0

Commit message: [jvrc1.urdf] Fix upper/lower limits of gripper mimic joints.

File: jvrc_description/urdf/jvrc1.urdf (robot description, URDF)
Before this commit: robot jvrc1, 60 links, 59 joints
Joints:
- joint L_LINDEX: limit lower=-1.57079632679 upper=0.0 effort=100.0 velocity=5.75958 -> lower=-2.356194490191 upper=2.356194490191 effort=100.0 velocity=5.75958
- joint L_LLITTLE: limit lower=-1.57079632679 upper=0.0 effort=100.0 velocity=5.75958 -> lower=-2.356194490191 upper=2.356194490191 effort=100.0 velocity=5.75958
- joint L_LTHUMB: limit lower=-0.0 upper=1.57079632679 effort=100.0 velocity=13.6135 -> lower=-2.356194490191 upper=2.356194490191 effort=100.0 velocity=13.6135
- joint L_UINDEX: limit lower=-1.57079632679 upper=0.0 effort=100.0 velocity=9.42477 -> lower=-0.785398163397 upper=0.785398163397 effort=100.0 velocity=9.42477
- joint L_ULITTLE: limit lower=-1.57079632679 upper=0.0 effort=100.0 velocity=9.42477 -> lower=-0.785398163397 upper=0.785398163397 effort=100.0 velocity=9.42477
- joint R_LINDEX: limit lower=0.0 upper=1.57079632679 effort=100.0 velocity=5.75958 -> lower=-2.356194490191 upper=2.356194490191 effort=100.0 velocity=5.75958
- joint R_LLITTLE: limit lower=0.0 upper=1.57079632679 effort=100.0 velocity=5.75958 -> lower=-2.356194490191 upper=2.356194490191 effort=100.0 velocity=5.75958
- joint R_LTHUMB: limit lower=-1.57079632679 upper=0.0 effort=100.0 velocity=13.6135 -> lower=-2.356194490191 upper=2.356194490191 effort=100.0 velocity=13.6135
- joint R_UINDEX: limit lower=0.0 upper=1.57079632679 effort=100.0 velocity=9.42477 -> lower=-0.785398163397 upper=0.785398163397 effort=100.0 velocity=9.42477
- joint R_ULITTLE: limit lower=0.0 upper=1.57079632679 effort=100.0 velocity=9.42477 -> lower=-0.785398163397 upper=0.785398163397 effort=100.0 velocity=9.42477

Commit message: Make the gripper limits coherent

File: jvrc_description/urdf/jvrc1.urdf (robot description, URDF)
Before this commit: robot jvrc1, 60 links, 59 joints
Joints:
- joint L_LINDEX: limit lower=-1.57079632679 upper=0.0 effort=100.0 velocity=5.75958 -> lower=-2.356194490191 upper=2.356194490191 effort=300.0 velocity=20.42034
- joint L_LLITTLE: limit lower=-1.57079632679 upper=0.0 effort=100.0 velocity=5.75958 -> lower=-2.356194490191 upper=2.356194490191 effort=300.0 velocity=20.42034
- joint L_LTHUMB: limit lower=-0.0 upper=1.57079632679 effort=100.0 velocity=13.6135 -> lower=-2.356194490191 upper=2.356194490191 effort=300.0 velocity=20.42034
- joint L_UINDEX: limit lower=-1.57079632679 upper=0.0 effort=100.0 velocity=9.42477 -> lower=-0.785398163397 upper=0.785398163397 effort=100.0 velocity=6.80678
- joint L_ULITTLE: limit lower=-1.57079632679 upper=0.0 effort=100.0 velocity=9.42477 -> lower=-0.785398163397 upper=0.785398163397 effort=100.0 velocity=6.80678
- joint R_LINDEX: limit lower=0.0 upper=1.57079632679 effort=100.0 velocity=5.75958 -> lower=-2.356194490191 upper=2.356194490191 effort=300.0 velocity=20.42034
- joint R_LLITTLE: limit lower=0.0 upper=1.57079632679 effort=100.0 velocity=5.75958 -> lower=-2.356194490191 upper=2.356194490191 effort=300.0 velocity=20.42034
- joint R_LTHUMB: limit lower=-1.57079632679 upper=0.0 effort=100.0 velocity=13.6135 -> lower=-2.356194490191 upper=2.356194490191 effort=300.0 velocity=20.42034
- joint R_UINDEX: limit lower=0.0 upper=1.57079632679 effort=100.0 velocity=9.42477 -> lower=-0.785398163397 upper=0.785398163397 effort=100.0 velocity=6.80678
- joint R_ULITTLE: limit lower=0.0 upper=1.57079632679 effort=100.0 velocity=9.42477 -> lower=-0.785398163397 upper=0.785398163397 effort=100.0 velocity=6.80678
